File: KiCad-template.kicad_pcb (KiCad board)
At the start: 2 copper layers, 28.8 x 18.8 mm, 1 part, among them J1 usb_c_12402012E212A

Commit message: [NEW] Added component for ESP32 5V Lion battery alimentation
Parts:
- removed J1: usb_c_12402012E212A, custom_library:usb_c_AMPHENOL_12402012E212A
Other:
- board outline removed
